File: main_controller2.kicad_sch (KiCad schematic)
At the start: 77 parts, among them J1 xt30, J10 Conn_01x04, J11 Conn_01x04, J12 Conn_01x04, J13 Conn_01x04, J2 Conn_01x04, J3 xt30, J4 Conn_01x08, J8 SMA, J9 Conn_01x04, Q1 FDN359BN, SW1 SW_SPST, SW2 SW_SPST, U1 ESP32-WROOM-32D, U10 BTN7030-1EPA, U11 PCA9557PW, U12 RFM95W-915S2, U13 W25N02KVZEIR, U14 MCP2517FD-xSL, U15 SN65HVD230, U2 BMI088, U3 china_buck_converter, U4 AP7361-33ER-13, U5 MS5611-01BA, U6 BTS70802, U7 BTN7030-1EPA, U8 BTN7030-1EPA, U9 BTN7030-1EPA, Y1 40MHz

Commit message: stackable version
Parts:
- removed C15: 0.1u, Capacitor_SMD:C_0603_1608Metric, symbol Device:C_Small
- removed J10, J11, J12, J13, J2, J9: Conn_01x04, Connector_JST:JST_XH_B4B-XH-A_1x04_P2.50mm_Vertical, symbol Connector_Generic:Conn_01x04
- removed J4: Conn_01x08, TerminalBlock_RND:TerminalBlock_RND_205-00007_1x08_P5.00mm_Horizontal, symbol Connector_Generic:Conn_01x08
- removed J8: SMA, Connector_Coaxial:SMA_Molex_73251-1153_EdgeMount_Horizontal, symbol Connector:Conn_Coaxial_x2_Isolated
- removed J?: Conn_01x25, symbol Connector_Generic:Conn_01x25
- removed J?: Conn_01x12, symbol Connector_Generic:Conn_01x12
- removed JP3, JP4: SolderJumper_2_Open, Jumper:SolderJumper-2_P1.3mm_Open_TrianglePad1.0x1.5mm, symbol Jumper:SolderJumper_2_Open
- removed U1: ESP32-WROOM-32D, RF_Module:ESP32-WROOM-32, symbol RF_Module:ESP32-WROOM-32D
- removed U12: RFM95W-915S2, RF_Module:HOPERF_RFM9XW_SMD, symbol RF_Module:RFM95W-915S2
- added J10: Conn_01x15, Connector_PinHeader_2.54mm:PinHeader_1x15_P2.54mm_Vertical, symbol Connector_Generic:Conn_01x15
- added J4, J6, J7, J8: Conn_01x02, Connector_JST:JST_XH_S2B-XH-A_1x02_P2.50mm_Horizontal, symbol Connector_Generic:Conn_01x02
- added J9: Conn_01x16, Connector_PinHeader_2.54mm:PinHeader_1x16_P2.54mm_Vertical, symbol Connector_Generic:Conn_01x16
- added R11, R12: 2k2, Resistor_SMD:R_0603_1608Metric, symbol Device:R_Small
- added U1: ESP32-PICO-MINI-02, lib:MODULE_ESP32-PICO-MINI-02U, symbol pico:ESP32-PICO-MINI-02
- C5: value big -> edda_cap
- D1, D2: footprint LED_SMD:LED_WS2812B_PLCC4_5.0x5.0mm_P3.2mm -> LED_SMD:LED_WS2812B-2020_PLCC4_2.0x2.0mm
- JP1: footprint Connector_JST:JST_XH_B2B-XH-A_1x02_P2.50mm_Vertical -> Connector_JST:JST_XH_S2B-XH-A_1x02_P2.50mm_Horizontal
- JP2: footprint Connector_AMASS:AMASS_XT30UPB-F_1x02_P5.0mm_Vertical -> Connector_AMASS:AMASS_XT30PW-F_1x02_P2.50mm_Horizontal
- U13: footprint Package_SO:SOIC-8_5.275x5.275mm_P1.27mm -> lib:SON127P800X600X80-9N-D
Connections:
- net BUZZER is gone; now on net BOOTLOADER: Q1.1 (G)
- net LORA_RESET is gone; now on net EDDA_EN: U11.10 (IO3)
- net +3V3: now also D1.1 (VDD), D2.1 (VDD), U14.14 (VDD), U15.5 (Vref), R11.2, R12.2, U1.3 (3V3)
- net +5V: now also C9.2; no longer C9.1, D1.1 (VDD), D2.1 (VDD)
- net 3V3: now also J10.5 (Pin_5)
- net 5V: now also J10.11 (Pin_11)
- net BOOTLOADER: now also U1.23 (IO0)
- net CAN_CS: now also U1.35 (IO21)
- net CAN_H: now also J10.10 (Pin_10)
- net CAN_IRQ: now also U1.7 (I39)
- net CAN_L: now also J10.9 (Pin_9)
- net CURR_EN: no longer U11.11 (IO4)
- net CURR_SEL: now also U11.11 (IO4); no longer U11.13 (IO6)
- net CURR_SENSE: now also U1.6 (I38)
- net EDDA_EN: no longer U11.12 (IO5)
- net Earth: now also C9.1, U14.7 (VSS), J4.1 (Pin_1), J6.1 (Pin_1), J7.1 (Pin_1), J8.1 (Pin_1), U1.1 (GND), U1.11 (GND), U1.14 (GND), U1.2 (GND), U1.36 (GND), U1.37 (GND), U1.38 (GND), U1.39 (GND), U1.40 (GND), U1.41 (GND), U1.42 (GND), U1.43 (GND), U1.44 (GND), U1.45 (GND), U1.46 (GND), U1.47 (GND), U1.48 (GND), U1.49 (GND), U1.50 (GND), U1.51 (GND), U1.52 (GND), U1.53 (GND), U1.54 (GND), U1.55 (GND), U1.56 (GND), U1.57 (GND), U1.58 (GND), U1.59 (GND), U1.60 (GND), U1.61 (GND); no longer C9.2
- net FLASH_CS: now also U1.34 (IO22)
- net GND: now also J10.1 (Pin_1), J10.14 (Pin_14), J10.15 (Pin_15), J10.2 (Pin_2), J10.8 (Pin_8), J9.1 (Pin_1), J9.12 (Pin_12), J9.16 (Pin_16), J9.8 (Pin_8)
- net HSPI_MISO: now also U14.12 (SDO), U1.19 (IO12)
- net HSPI_MOSI: now also U14.11 (SDI), U1.20 (IO13)
- net HSPI_SCK: now also U14.10 (SCK), U1.18 (IO14)
- net PYRO_1: now also J4.2 (Pin_2), U1.33 (IO19)
- net PYRO_2: now also J6.2 (Pin_2), U1.26 (IO20)
- net PYRO_3: now also J7.2 (Pin_2)
- net PYRO_4: now also J8.2 (Pin_2)
- net RX1: now also J9.4 (Pin_4), U1.10 (I35)
- net RX2: now also J9.6 (Pin_6), U1.9 (I34)
- net SCL: no longer R7.1
- net SDA: no longer R6.1
- net TX1: now also J9.5 (Pin_5), U1.12 (IO32)
- net TX2: now also J9.7 (Pin_7), U1.13 (IO33)
- net VBAT_SENSE: now also U1.5 (I37)
- net VCC: now also J10.12 (Pin_12), J10.13 (Pin_13), J10.3 (Pin_3), J10.4 (Pin_4)
- net VSPI_MISO: now also J9.10 (Pin_10), U1.4 (I36); no longer U14.12 (SDO)
- net VSPI_MOSI: now also J9.9 (Pin_9), U1.27 (IO7); no longer U14.11 (SDI)
- net VSPI_SCK: now also J9.11 (Pin_11), U1.28 (IO8); no longer U14.10 (SCK)
- net at R8.2, SW2.2 (B): now also U1.8 (EN)
- net CAN_MISC_PIN: no longer names the net of U11.14 (IO7)
- net CAN_MISC_PIN: no longer U15.5 (Vref)
- new net: U1.25 (NC), U1.32 (NC)
- new net LED_RMT: U1.15 (IO25)
- new net MISC_GPIO0: J9.13 (Pin_13)
- new net MISC_GPIO1: J9.14 (Pin_14)
- new net MISC_GPIO2: J9.15 (Pin_15)
- new net MISC_IO0: U1.29 (IO5)
- new net MISC_IO1: U1.21 (IO15)
- new net MISC_IO2: U11.12 (IO5)
- new net MISC_IO3: U11.13 (IO6)
- new net RX0: J9.2 (Pin_2), U1.30 (RXD0)
- new net SCL0: R7.1, U1.24 (IO4)
- new net SCL1: J10.6 (Pin_6), R12.1, U1.17 (IO27)
- new net SDA0: R6.1, U1.22 (IO2)
- new net SDA1: J10.7 (Pin_7), R11.1, U1.16 (IO26)
- new net TX0: J9.3 (Pin_3), U1.31 (TXD0)
- no-connect marks 25 -> 15
Other:
- note added: "direct"
- note removed: "Free up pins for another I2C? sacrifice GPS2 tx?"
- note removed: "LORA"
- note removed: "connectors"
- note removed: "way to bypass the controller? probably not useful"
- moved on the sheet: C14, C4, C8, D2, R6, R7, R8, SW1, SW2, U11

Commit message: move to esp pico
Parts:
- removed R9: 300, Resistor_SMD:R_0603_1608Metric, symbol Device:R_Small
- removed U1: ESP32-PICO-MINI-02, lib:MODULE_ESP32-PICO-MINI-02U, symbol pico:ESP32-PICO-MINI-02
- added C15: 0.1u, Capacitor_SMD:C_0603_1608Metric, symbol Device:C_Small
- added C?: 4.7u, Capacitor_SMD:C_0603_1608Metric, symbol Device:C_Small
- added R9: R, Resistor_SMD:R_1206_3216Metric_Pad1.30x1.75mm_HandSolder, symbol Device:R
- added U1: ESP32-PICO-D4, Package_DFN_QFN:QFN-48-1EP_7x7mm_P0.5mm_EP5.3x5.3mm, symbol RF_Module:ESP32-PICO-D4
- added U12: INA219AxD, Package_SO:SOIC-8_3.9x4.9mm_P1.27mm, symbol Analog_ADC:INA219AxD
- D1, D2: footprint LED_SMD:LED_WS2812B-2020_PLCC4_2.0x2.0mm -> LED_SMD:LED_WS2812B_PLCC4_5.0x5.0mm_P3.2mm
Connections:
- net SCL is gone; now on net SCL0: U11.1 (SCL), U2.8 (SCL/SCK), U5.8 (SCLK)
- net SDA is gone; now on net SDA0: U11.2 (SDA), U2.9 (SDA/SDI), U5.7 (SDI/SDA)
- net +3V3: now also C15.1, C?.1, U1.1 (VDDA), U1.19 (VDD3P3_RTC), U1.26 (VDD_SDIO), U1.3 (VDDA3P3), U1.37 (VDD3P3_CPU), U1.4 (VDDA3P3), U1.43 (VDDA), U1.46 (VDDA), U12.5 (VS)
- net +BATT: now also R9.2, U12.7 (IN-); no longer J1.2, R1.1
- net BOOTLOADER: now also U1.23 (IO0); no longer Q1.1 (G)
- net CAN_CS: now also U1.38 (IO19)
- net CAN_IRQ: now also U1.11 (IO35)
- net CURR_SENSE: now also U1.7 (SENSOR_CAPN); no longer U6.4 (IS)
- net Earth: now also C15.2, C?.2, U12.1 (A1), U12.2 (A0), U12.6 (GND)
- net FLASH_CS: now also U1.42 (IO21)
- net HSPI_MISO: now also U1.18 (IO12)
- net HSPI_MOSI: now also U1.20 (IO13)
- net HSPI_SCK: now also U1.17 (IO14)
- net LED_RMT: now also U1.39 (IO22)
- net MISC_IO0: now also U1.22 (IO2), U1.24 (IO4)
- net MISC_IO1: now also U1.29 (SD3/IO10)
- net PYRO_1: now also U1.21 (IO15)
- net PYRO_2: now also U1.35 (IO18)
- net RX0: now also U1.40 (U0RXD/IO3)
- net RX1: now also U1.6 (SENSOR_CAPP)
- net RX2: now also U1.5 (SENSOR_VP)
- net SCL0: now also U1.13 (IO33), U12.4 (SCL)
- net SCL1: now also U1.14 (IO25)
- net SDA0: now also U1.12 (IO32), U12.3 (SDA)
- net SDA1: now also U1.36 (IO23)
- net TX0: now also U1.41 (U0TXD/IO1)
- net TX1: now also U1.15 (IO26)
- net TX2: now also U1.16 (IO27)
- net VBAT_SENSE: now also U1.8 (SENSOR_VN)
- net VSPI_MISO: now also U1.10 (IO34)
- net VSPI_MOSI: now also U1.34 (IO5)
- net VSPI_SCK: now also U1.28 (SD2/IO9)
- net at R8.2, SW2.2 (B): now also U1.9 (EN)
- net CURR_EN: no longer names the net of U6.3 (DEN)
- net CURR_SEL: no longer names the net of U6.5 (DSEL)
- net CURR_SEL: no longer U11.11 (IO4)
- new net: J1.2, R1.1, R9.1, U12.8 (IN+)
- new net BUZZER: Q1.1 (G)
- no-connect marks 15 -> 25
Other:
- note added: "CURRENT SENSE"
- note added: "INPUT ONLY"
- note added: "LOGIC LEVEL"
- note added: "POWER MANAGEMENT"
- note removed: "300 seems a bit low"
- moved on the sheet: C1, C14, C16, C17, C2, C3, C4, C5, C6, C7, J1, J3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
